File: Hardware/monkey_arduino_shield/monkey_arduino_shield.kicad_pcb (KiCad board)
At the start: 2 copper layers, 68.6 x 53.3 mm, 8 parts, among them P1 Power, P2 Analog, P3 Digital, P4 Digital, P5 CONN_01X01, P6 CONN_01X01, P7 CONN_01X01, P8 CONN_01X01

Commit message: First Hardware Rev
Added RAM, motor drivers, audio I/O
Parts:
- added C1: 1u, Capacitor_SMD:C_1206_3216Metric, F.Cu at (139.8, 118.6)
- added C2: 1u, Capacitor_SMD:C_1206_3216Metric, F.Cu at (139.7, 113.3)
- added J1: Speaker_OUT, TerminalBlock:TerminalBlock_bornier-2_P5.08mm, F.Cu at (115.7, 114.4)
- added J3: Screw_Terminal_01x03, TerminalBlock:TerminalBlock_bornier-3_P5.08mm, F.Cu at (170.3, 98.4)
- added J4: Screw_Terminal_01x03, TerminalBlock:TerminalBlock_bornier-3_P5.08mm, F.Cu at (170.3, 81.0)
- added J5: MIC_IN, TerminalBlock:TerminalBlock_bornier-3_P5.08mm, F.Cu at (115.7, 103.3)
- added R1: 10K, Resistor_SMD:R_0603_1608Metric, F.Cu at (126.2, 118.9)
- added R2: 150k, Resistor_SMD:R_0603_1608Metric, F.Cu at (131.8, 118.6)
- added R3: 150k, Resistor_SMD:R_0603_1608Metric, F.Cu at (131.9, 114.3)
- added U1: W25Q128JVS, Package_SO:SOIC-8_5.23x5.23mm_P1.27mm, F.Cu at (128.8, 82.8)
- added U2: SN74LVC2T45DCUR, Package_SO:VSSOP-8_2.4x2.1mm_P0.5mm, F.Cu at (142.7, 84.3)
- added U3: SN74LVC2T45DCUR, Package_SO:VSSOP-8_2.4x2.1mm_P0.5mm, F.Cu at (142.7, 81.3)
- added U4: TPA2005D1DRB, Package_SO:MSOP-8-1EP_3x3mm_P0.65mm_EP1.68x1.88mm, F.Cu at (124.1, 115.4)
Connections:
- P3 pad 1: /A5(SCL) -> /A5(SCL_)
- P3 pad 2: /A4(SDA) -> /A4(SDA_)
- P3 pad 5: /13(SCK) -> /13(HV_SCK)
- P3 pad 6: /12(MISO) -> /12(HV_MISO)
- P3 pad 7: /11(**/MOSI) -> /11(HV_MOSI)
Routing:
- net GND: track 0.00 -> 169.3 mm, vias 0 -> 3
- net +5V: track 0.00 -> 118.4 mm, vias 0 -> 2
- net +3V3: track 0.00 -> 95.9 mm, vias 0 -> 3
- net /A0: track 0.00 -> 60.2 mm
- net /LV_MOSI: track 0.00 -> 36.1 mm, vias 0 -> 2
- net /6(**): track 0.00 -> 32.5 mm
- net /LV_SCK: track 0.00 -> 30.4 mm
- net /A1: track 0.00 -> 29.1 mm, vias 0 -> 3
- net /13(HV_SCK): track 0.00 -> 22.6 mm
- net /11(HV_MOSI): track 0.00 -> 18.9 mm, vias 0 -> 2
- net /5(**): track 0.00 -> 14.1 mm
- net /12(HV_MISO): track 0.00 -> 10.1 mm, vias 0 -> 2
- net /LV_MISO: track 0.00 -> 9.82 mm
- net Net-(J1-Pad1): track 0.00 -> 6.27 mm
- net Net-(R2-Pad1): track 0.00 -> 6.14 mm
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- added copper zone on B.Cu, net GND
