File: Hardware/monkey_arduino_shield/monkey_arduino_shield.sch (KiCad schematic (older format))
At the start: 8 parts, among them P1 Power, P2 Analog, P3 Digital, P4 Digital, P5 CONN_01X01, P6 CONN_01X01, P7 CONN_01X01, P8 CONN_01X01

Commit message: First Hardware Rev
Added RAM, motor drivers, audio I/O
Parts:
- added C1, C2: 1u, Capacitor_SMD:C_1206_3216Metric, symbol Device:C_Small
- added J1: Speaker_OUT, TerminalBlock:TerminalBlock_bornier-2_P5.08mm, symbol Connector:Screw_Terminal_01x02
- added J3, J4: Screw_Terminal_01x03, TerminalBlock:TerminalBlock_bornier-3_P5.08mm, symbol Connector:Screw_Terminal_01x03
- added J5: MIC_IN, TerminalBlock:TerminalBlock_bornier-3_P5.08mm, symbol Connector:Screw_Terminal_01x03
- added R1: 10K, Resistor_SMD:R_0603_1608Metric, symbol Device:R_Small
- added R2, R3: 150k, Resistor_SMD:R_0603_1608Metric, symbol Device:R_Small
- added U1: W25Q128JVS, Package_SO:SOIC-8_5.23x5.23mm_P1.27mm, symbol Memory_Flash:W25Q128JVS
- added U2, U3: SN74LVC2T45DCUR, Package_SO:VSSOP-8_2.4x2.1mm_P0.5mm, symbol Logic_LevelTranslator:SN74LVC2T45DCUR
- added U4: TPA2005D1DRB, Package_SO:MSOP-8-1EP_3x3mm_P0.65mm_EP1.68x1.88mm, symbol SparkFun-AnalogIC:TPA2005D1DRB
Connections:
- net +3V3: now also J5.1 (Pin_1), U1.1 (~CS), U1.8 (VCC), U2.1 (VCCA), U3.1 (VCCA), U3.5 (DIR)
- net +5V: now also J3.3 (Pin_3), J4.3 (Pin_3), R1.1, U2.8 (VCCB), U3.8 (VCCB), U4.6 (VDD)
- net 5(**): now also J4.2 (Pin_2)
- net 6(**): now also J3.2 (Pin_2)
- net A0: now also J5.3 (Pin_3)
- net A1: now also C1.2
- net A4(SDA): no longer P3.2 (Pin_2)
- net A5(SCL): no longer P3.1 (Pin_1)
- net GND: now also C2.1, J1.2 (Pin_2), J3.1 (Pin_1), J4.1 (Pin_1), J5.2 (Pin_2), U1.4 (GND), U2.4 (GND), U2.5 (DIR), U3.4 (GND), U4.10 (GND), U4.11 (GND), U4.12 (GND), U4.13 (GND), U4.7 (GND), U4.8 (OUT-), U4.9 (GND)
- net 11(**/MOSI) renamed 11(HV_MOSI)
- net 11(HV_MOSI): now also U2.7 (B1)
- net 12(MISO) renamed 12(HV_MISO)
- net 12(HV_MISO): now also U3.7 (B1)
- net 13(SCK) renamed 13(HV_SCK)
- net 13(HV_SCK): now also U2.6 (B2)
- new net: R1.2, U4.1 (SHUTDOWN)
- new net: R2.1, U4.3 (IN+)
- new net: R3.1, U4.4 (IN-)
- new net: J1.1 (Pin_1), U4.5 (OUT+)
- new net: C1.1, R2.2
- new net: C2.2, R3.2
- new net A4(SDA_): P3.2 (Pin_2)
- new net A5(SCL_): P3.1 (Pin_1)
- new net LV_MISO: U1.2 (DO(IO1)), U3.2 (A1)
- new net LV_MOSI: U1.5 (DI(IO0)), U2.2 (A1)
- new net LV_SCK: U1.6 (CLK), U2.3 (A2)
- no-connect marks 5 -> 9
Other:
- note added: "MICROPHONE INPUT (PREAMPLIFIED)"
- note added: "MOTOR CONNECTIONS"
- note added: "SPI LEVEL SHIFT (5V -> 3.3V)"
- note added: "SRAM EXPANSION"
